File: schematic/calculator.kicad_pcb (KiCad board)
At the start: 2 copper layers, 62 x 42 mm, 27 parts, among them J1 PinHeader_1x04_P2.54mm_Vertic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, SW1 SW_PUSH_6mm, SW10 SW_PUSH_6mm, SW11 SW_PUSH_6mm, SW12 SW_PUSH_6mm, SW13 SW_PUSH_6mm, SW14 SW_PUSH_6mm, SW15 SW_PUSH_6mm, SW16 SW_PUSH_6mm, SW2 SW_PUSH_6mm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

Commit message: Add OLED header connector to PCB schematic
Parts:
- added OLED1: PinHeader_1x04_P2.54mm_Vertical, Connector_PinHeader_2.54mm:PinHeader_1x04_P2.54mm_Vertical, F.Cu at (31.0, 14.0)
Routing:
- net I2C_SCL: track 0.00 -> 20.9 mm
- net I2C_SDA: track 0.00 -> 12.3 mm
- net GND: track 11.0 -> 13.0 mm
- net +3.3V: track 91.0 -> 93.0 mm
Changed lines of the file:
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@@
 	(net 17 "SWDIO")
 	(net 18 "SWCLK")
+	(net 19 "I2C_SCL")
+	(net 20 "I2C_SDA")
 	(gr_line
 		(start 0 0)
@@
 		(property "Value" "SW_PUSH_6mm"
 			(at 42 31.05 0)
+			(layer "F.Fab")
+			(effects
+				(font
+					(size 1.27 1.27)
+				)
+			)
+		)
+		(property "Datasheet" ""
+			(at 0 0 0)
+			(layer "F.Fab")
+			(hide yes)
+			(effects
+				(font
+					(size 1.27 1.27)
+				)
+			)
+		)
+		(property "Description" ""
+			(at 0 0 0)
+			(layer "F.Fab")
+			(hide yes)
+			(effects
+				(font
+					(size 1.27 1.27)
+				)
+			)
+		)
+		(duplicate_pad_numbers_are_jumpers no)
+		(embedded_fonts no)
+	)
+	(footprint "Connector_PinHeader_2.54mm:PinHeader_1x04_P2.54mm_Vertical"
+		(layer "F.Cu")
+		(at 31 14)
+		(property "Reference" "OLED1"
+			(at 31 13.95 0)
+			(layer "F.SilkS")
+			(effects
+				(font
+					(size 1 1)
+					(thickness 0.15)
+				)
+			)
+		)
+		(property "Value" "PinHeader_1x04_P2.54mm_Vertical"
+			(at 31 14.05 0)
 			(layer "F.Fab")
 			(effects
@@
 	(segment (start 55 35.73) (end 57 35.73) (width 0.25) (layer "F.Cu") (net 1))
 	(segment (start 55 33.19) (end 57 33.19) (width 0.25) (layer "F.Cu") (net 0))
+	(segment (start 28.25 3.1) (end 31.25 3.1) (width 0.25) (layer "F.Cu") (net 19))
+	(segment (start 31.25 3.1) (end 27 3.1) (width 0.25) (layer "F.Cu") (net 19))
+	(segment (start 27 3.1) (end 27 12.73) (width 0.25) (layer "F.Cu") (net 19))
+	(segment (start 27 12.73) (end 31 12.73) (width 0.25) (layer "F.Cu") (net 19))
+	(segment (start 27.1 7.75) (end 24.1 7.75) (width 0.25) (layer "F.Cu") (net 20))
+	(segment (start 24.1 7.75) (end 25 7.75) (width 0.25) (layer "F.Cu") (net 20))
+	(segment (start 25 7.75) (end 25 10.19) (width 0.25) (layer "F.Cu") (net 20))
+	(segment (start 25 10.19) (end 31 10.19) (width 0.25) (layer "F.Cu") (net 20))
+	(segment (start 31 17.81) (end 29 17.81) (width 0.25) (layer "F.Cu") (net 0))
+	(segment (start 31 15.27) (end 33 15.27) (width 0.25) (layer "F.Cu") (net 1))
 	(segment (start 30.75 3.1) (end 31.75 3.1) (width 0.25) (layer "F.Cu") (net 1))
 	(segment (start 27.1 5.75) (end 28.1 5.75) (width 0.25) (layer "F.Cu") (net 1))
